Commit message: GT: fixed bugs

File: urdf/sensors/kinetic_rgbd.urdf.xacro (robot description, xacro)
@@ -31,5 +31,5 @@
                 <box size="0.06 0.1 0.03" />
                     -->
-                    <mesh filename="package://ur_app_youtube/meshes/sensors/camera/kinetic.stl"/>
+                    <mesh filename="package://pose_estimation/meshes/sensors/camera/kinetic.stl"/>
                 </geometry>
                 <material name="DarkGrey"/>
@@ -37,5 +37,5 @@
             <collision>
                 <geometry>
-                    <mesh filename="package://ur_app_youtube/meshes/sensors/camera/kinetic.dae"/>
+                    <mesh filename="package://pose_estimation/meshes/sensors/camera/kinetic.dae"/>
                 </geometry>
             </collision>

File: urdf/ur5_cam.xacro (robot description, xacro)
@@ -5,4 +5,5 @@
 <!-- =================================================================================== -->
 <robot name="ur5_robot" xmlns:xacro="http://ros.org/wiki/xacro">
+    <xacro:property name="deg_to_rad" value="0.017453292519943295"/> <!-- pi/180 -->
     <!-- Include the table definition from another file -->
     <xacro:include filename="$(find pose_estimation)/urdf/table.urdf.xacro"/>
