Commit message: adjusted final problems

File: pose_estimation/urdf/ur5_cam.xacro (robot description, xacro)
@@ -99,5 +99,5 @@
         <parent link="world"/>
         <child link="table"/>
-        <origin xyz="0 0 0" rpy="0 0 0"/> <!-- Adjust this to half the table thickness -->
+        <origin xyz="0 0 0.05" rpy="0 0 0"/> <!-- Adjust this to half the table thickness -->
     </joint>
     <!-- Now attach the robot to the table. -->
@@ -110,5 +110,5 @@
              Adjust as needed based on how the meshes align.
         -->
-        <origin xyz="0 0 0.05" rpy="0 0 0"/>
+        <origin xyz="0 0 0" rpy="0 0 0"/>
     </joint>
     <link name="shoulder_link">

File: robotiq_description/urdf/robotiq_85_gripper.urdf.xacro (robot description, xacro)
@@ -81,10 +81,10 @@
             </inertial>
         </link>
-        <joint name="${prefix}robotiq_85_left_finger_joint" type="fixed">
+        <joint name="${prefix}robotiq_85_left_finger_joint" type="continuous">
             <parent link="${prefix}robotiq_85_left_knuckle_link"/>
             <child link="${prefix}robotiq_85_left_finger_link"/>
             <origin xyz="-0.00408552455 -0.03148604435 0.0" rpy="0 0 0" />
         </joint>
-        <joint name="${prefix}robotiq_85_right_finger_joint" type="fixed">
+        <joint name="${prefix}robotiq_85_right_finger_joint" type="continuous">
             <parent link="${prefix}robotiq_85_right_knuckle_link"/>
             <child link="${prefix}robotiq_85_right_finger_link"/>

Commit message: final adjustments

File: pose_estimation/urdf/ur5_cam.xacro (robot description, xacro)
@@ -99,5 +99,5 @@
         <parent link="world"/>
         <child link="table"/>
-        <origin xyz="0 0 0.05" rpy="0 0 0"/> <!-- Adjust this to half the table thickness -->
+        <origin xyz="0 0 0" rpy="0 0 0"/> <!-- Adjust this to half the table thickness -->
     </joint>
     <!-- Now attach the robot to the table. -->
@@ -110,5 +110,5 @@
              Adjust as needed based on how the meshes align.
         -->
-        <origin xyz="0 0 0" rpy="0 0 0"/>
+        <origin xyz="0 0 0.05" rpy="0 0 0"/>
     </joint>
     <link name="shoulder_link">
