Commit message: turned topics to services, added color to spawn objects, changed spawn objects, added new launch file, added gitignore,

File: pose_estimation/urdf/cylinder.urdf (robot description, URDF)
Before this commit: robot cylinder, 1 links, 0 joints
Links:
- link cylinder_link: geometry collision cylinder length=0.1 radius=0.025; visual cylinder length=0.1 radius=0.025

Commit message: added pick and place motion, changed material of cylinder

File: pose_estimation/urdf/cylinder.urdf (robot description, URDF)
Before this commit: robot cylinder, 1 links, 0 joints
Links:
- link cylinder_link: mass 0.1 -> 0.2
